Commit message: fixing urdf...

File: resources/ur5/ur5_spherized.urdf (robot description, URDF)
Before this commit: robot ur5_robotiq85, 22 links, 21 joints
Links:
- link forearm_link: geometry collision sphere radius=0.05; collision sphere radius=0.05

Commit message: updated ur5 spherized

File: resources/ur5/ur5_spherized.urdf (robot description, URDF)
Before this commit: robot ur5_robotiq85, 22 links, 21 joints
Links:
- link forearm_link: geometry collision sphere radius=0.04; collision sphere radius=0.04
- link robotiq_85_left_finger_tip_link: geometry collision sphere radius=0.015; collision sphere radius=0.015
- link robotiq_85_right_finger_tip_link: geometry collision sphere radius=0.015; collision sphere radius=0.015
