Commit message: remove adjacent and never colliding frames from approximation, updated ur10e urdf to work

File: resources/ur10e/ur_10e_spherized.urdf (robot description, URDF)
Before this commit: robot ur10e-2f85, 22 links, 21 joints
Links:
- link upper_arm_link: geometry collision sphere radius=0.10; collision sphere radius=0.10
Joints:
- joint shoulder_lift_joint: limit lower=-6.283185307179586 upper=6.283185307179586 effort=330.0 velocity=2.0943951023931953 -> lower=-3.141592653589793 upper=3.141592653589793 effort=330.0 velocity=2.0943951023931953
- joint shoulder_pan_joint: limit lower=-6.283185307179586 upper=6.283185307179586 effort=330.0 velocity=2.0943951023931953 -> lower=-3.141592653589793 upper=3.141592653589793 effort=330.0 velocity=2.0943951023931953
- joint wrist_1_joint: limit lower=-6.283185307179586 upper=6.283185307179586 effort=54.0 velocity=3.141592653589793 -> lower=-3.141592653589793 upper=3.141592653589793 effort=54.0 velocity=3.141592653589793
- joint wrist_2_joint: limit lower=-6.283185307179586 upper=6.283185307179586 effort=54.0 velocity=3.141592653589793 -> lower=-3.141592653589793 upper=3.141592653589793 effort=54.0 velocity=3.141592653589793
- joint wrist_3_joint: limit lower=-6.283185307179586 upper=6.283185307179586 effort=54.0 velocity=3.141592653589793 -> lower=-3.141592653589793 upper=3.141592653589793 effort=54.0 velocity=3.141592653589793
