Commit message: yey better

File: resources/a200_1044/a200_1044_spherized.urdf (robot description, URDF)
Before this commit: robot a200_1044, 50 links, 49 joints
Links:
- link base_link: geometry collision sphere radius=0.104531; collision sphere radius=0.105393
- link link1: geometry collision sphere radius=0.072497; collision sphere radius=0.078856
- link rig_link: geometry collision sphere radius=0.160061; collision sphere radius=0.160285
- link top_plate_link: geometry visual mesh filename=meshes/clearpath_platform_description/meshes/a200/attachmen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
